Commit message: adding all local changes

File: rby1_description/urdf/rby1.ros2_control.xacro (robot description, xacro)
@@ -11,14 +11,16 @@
             <!-- joint: wheel -->
             <joint name="right_wheel">
-                <command_interface name="position"/>
+                <command_interface name="velocity"/>
                 <state_interface name="position">
                   <param name="initial_value">${initial_positions['right_wheel']}</param>
                 </state_interface>
+                <state_interface name="velocity"/>
             </joint>
             <joint name="left_wheel">
-                <command_interface name="position"/>
+                <command_interface name="velocity"/>
                 <state_interface name="position">
                   <param name="initial_value">${initial_positions['left_wheel']}</param>
                 </state_interface>
+                <state_interface name="velocity"/>
             </joint>
             <!-- joint: torso -->

File: rby1_description/urdf/rby1.urdf (robot description, URDF)
Before this commit: robot rby1, 35 links, 34 joints
Links:
- added link lidar_left_link, mass 0.125; collision cylinder length=0.055 radius=0.0508; visual cylinder length=0.055 radius=0.0508
- added link lidar_right_link, mass 0.125; collision cylinder length=0.055 radius=0.0508; visual cylinder length=0.055 radius=0.0508
- added link link_left_eef
- added link link_left_realsense
- added link link_right_eef
- added link link_right_realsense; collision box size=0.065 0.065 0.065
Joints:
- added joint left_eef: type fixed, parent link_left_arm_6, child link_left_eef, origin xyz=0.0 0.0 -0.2578 rpy=0.0 0.0 0.0
- added joint left_realsense: type fixed, parent link_left_arm_6, child link_left_realsense, origin xyz=0.0 0.053 -0.0243 rpy=0.0 0.0 0.0
- added joint lidar_left_joint: type fixed, parent base, child lidar_left_link, origin xyz=0.228 0.18 0.23 rpy=0 0 0.7854
- added joint lidar_right_joint: type fixed, parent base, child lidar_right_link, origin xyz=0.228 -0.18 0.23 rpy=0 0 -0.7854
- added joint right_eef: type fixed, parent link_right_arm_6, child link_right_eef, origin xyz=0.0 0.0 -0.2578 rpy=0.0 0.0 0.0
- added joint right_realsense: type fixed, parent link_right_arm_6, child link_right_realsense, origin xyz=0.0 -0.053 -0.0243 rpy=0.0 0.0 0.0
- joint left_arm_6: limit lower=-2.792526803 upper=2.792526803 effort=8.0 velocity=2.094395102 -> lower=-2.70 upper=2.70 effort=8.0 velocity=2.094395102
- joint right_arm_6: limit lower=-2.792526803 upper=2.792526803 effort=8.0 velocity=2.094395102 -> lower=-2.70 upper=2.70 effort=8.0 velocity=2.094395102
- joint world_to_base: type planar -> fixed

File: rby1_description/urdf/rby1.urdf.xacro (robot description, xacro)
@@ -4,5 +4,5 @@
     <xacro:arg name="robot_ip" default="" />
     <!-- Import rby1 urdf file -->
-    <xacro:include filename="$(find rby1_description)/urdf/rby1.urdf" />
+    <xacro:include filename="$(find rby1_description)/urdf/rby1_no_world.urdf" />
     <!-- Import control_xacro -->
     <xacro:include filename="$(find rby1_description)/urdf/rby1.ros2_control.xacro" />

File: rby1_moveit_config/config/rby1.urdf.xacro (robot description, xacro)
@@ -3,5 +3,5 @@
     <xacro:arg name="initial_positions_file" default="initial_positions.yaml" />
     <!-- Import rby1 urdf file -->
-    <xacro:include filename="$(find rby1_description)/urdf/rby1.urdf" />
+    <xacro:include filename="$(find rby1_description)/urdf/rby1_no_world.urdf" />
     <!-- Import control_xacro -->
     <xacro:include filename="rby1.ros2_control.xacro" />
