Commit message: fixed bad joint limits (`{left\right}_arm_4`)

File: rby1_description/urdf/rby1_no_world.urdf (robot description, URDF)
Before this commit: robot rby1, 40 links, 39 joints
Joints:
- joint left_arm_4: limit lower=-3.141592654 upper=3.141592654 effort=10.0 velocity=6.283185308 -> lower=-3.13 upper=3.13 effort=10.0 velocity=6.283185308
- joint right_arm_4: limit lower=-3.141592654 upper=3.141592654 effort=10.0 velocity=6.283185308 -> lower=-3.13 upper=3.13 effort=10.0 velocity=6.283185308

Commit message: update collision model(s) for realsense

File: rby1_description/urdf/rby1_no_world.urdf (robot description, URDF)
Before this commit: robot rby1, 40 links, 39 joints
Links:
- link link_left_realsense: geometry collision box size=0.120 0.065 0.065
- link link_right_realsense: geometry collision box size=0.120 0.065 0.065
